File: dome_center_pcb.kicad_pcb (KiCad board)
At the start: 4 copper layers, 100 x 114.9 mm, 97 parts, among them J1 350211-1, J2 Conn_01x14_Pin, J3 Conn_01x14_Pin, J4 Conn_01x14_Pin, J5 Conn_01x14_Pin, J6 Conn_01x14_Pin, J7 USB_B, U1 FT4232H, U10 DS2431P+T, U11 AMS1117-3.3, U2 USB2517-JZX-TR, U3 FT2232HL, U4 93LC56BT-I/OT, U5 93LC56BT-I/OT, U6 DS2431P+T, U7 DS2431P+T, U8 DS2431P+T, U9 DS2431P+T, X1 X322512MSB4SI, X2 X322512MSB4SI, Y1 Crystal

Commit message: Updating XML
Other:
- board text added: "https://github.com/daveismith/r2-warpcore-center <<hash>>"
Changed lines of the file:
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@@
   (gr_arc (start 100 51.154691) (mid 100.267949 50.154701) (end 100.999987 49.422647)
     (stroke (width 0.1) (type default)) (layer "Edge.Cuts"))
+  (gr_text "https://github.com/daveismith/r2-warpcore-center\n<<hash>>" (at 150.241 27.305 30) (layer "B.SilkS")
+    (effects (font (size 1.25 1.25) (thickness 0.3048) bold) (justify left bottom mirror))
+  )
   (gr_text "Saber Launcher" (at 173.3804 119.1006 210) (layer "F.SilkS")
     (effects (font (size 1.524 1.524) (thickness 0.3048) bold))

Commit message: Conversion to a simplified version.
Parts:
- removed C1, C18, C39, C41, C43, C45: 4.7uF, Resistor_SMD:R_0402_1005Metric
- removed C10, C11, C12, C13, C14, C15, C16, C17, C2, C21, C22, C23, C24, C26, C27, C28, C3, C30, C31, C32, C4, C5, C6, C7, C8, C9: 100nF, Capacitor_SMD:C_0402_1005Metric
- removed C19, C20, C25, C29, C33, C34: 1uF, Capacitor_SMD:C_0402_1005Metric
- removed C35, C36, C37, C38: 33pF, Resistor_SMD:R_0201_0603Metric
- removed C40, C42, C44, C46: 100nF, Resistor_SMD:R_0402_1005Metric
- removed C47, C50: 22uF, Capacitor_SMD:C_0805_2012Metric
- removed C48, C49: 10uF, Capacitor_SMD:C_0603_1608Metric
- removed C51, C52: 33pF, Capacitor_SMD:C_0402_1005Metric
- removed FB1, FB2, FB3, FB4: 600Ω@100MHz, Resistor_SMD:R_0603_1608Metric
- removed R1, R8: 12K, Resistor_SMD:R_0402_1005Metric
- removed R10: 330, Resistor_SMD:R_0402_1005Metric
- removed R11, R12: 100K, Resistor_SMD:R_0402_1005Metric
- removed R13, R15, R17, R19, R4, R6: 10K, Resistor_SMD:R_0402_1005Metric
- removed R14, R16, R18: R, Resistor_SMD:R_0402_1005Metric
- removed R2, R7: 1K, Resistor_SMD:R_0402_1005Metric
- removed R20: 1M, Resistor_SMD:R_0603_1608Metric
- removed R3, R5: 2K, Resistor_SMD:R_0402_1005Metric
- removed R9: 12K/1.0%, Resistor_SMD:R_0402_1005Metric
- removed U1: FT4232H, Package_QFP:LQFP-64_10x10mm_P0.5mm
- removed U10, U6, U7, U8, U9: DS2431P+T, easyeda2kicad:TSOC-6_L4.0-W4.0-P1.27-BL
- removed U11: AMS1117-3.3, Package_TO_SOT_SMD:SOT-223-3_TabPin2
- removed U2: USB2517-JZX-TR, easyeda2kicad:QFN-64_L9.0-W9.0-P0.50-BL-EP4.8
- removed U3: FT2232HL, easyeda2kicad:LQFP-64_L10.0-W10.0-P0.50-LS12.0-TL
- removed U4, U5: 93LC56BT-I/OT, easyeda2kicad:SOT-23-6_L2.9-W1.6-P0.95-LS2.8-BR
- removed X1, X2: X322512MSB4SI, easyeda2kicad:OSC-SMD_4P-L3.2-W2.5-BL
- removed Y1: Crystal, Crystal:Crystal_SMD_HC49-SD
- added J10: 171825-4, easyeda2kicad:HDR-TH_4P-P2.54-D1.0, F.Cu at (124.8, 111.8)
- added J11: 171825-4, easyeda2kicad:HDR-TH_4P-P2.54-D1.0, F.Cu at (184.1, 84.3)
- added J12: 171825-4, easyeda2kicad:HDR-TH_4P-P2.54-D1.0, F.Cu at (191.0, 84.3)
- added J13: Conn_01x07_Pin, Connector_JST:JST_XH_B7B-XH-A_1x07_P2.50mm_Vertical, F.Cu at (152.4, 31.5)
- added J8: 171825-4, easyeda2kicad:HDR-TH_4P-P2.54-D1.0, F.Cu at (134.2, 40.6)
- added J9: 171825-4, easyeda2kicad:HDR-TH_4P-P2.54-D1.0, F.Cu at (109.0, 73.4)
- J2, J3, J4, J5, J6: value Conn_01x14_Pin -> Conn_01x03_Pin; footprint Connector_JST:JST_XH_B14B-XH-A_1x14_P2.50mm_Vertical -> Connector_JST:JST_XH_B3B-XH-A_1x03_P2.50mm_Vertical
- J7: value USB_B -> Conn_01x05_Pin; footprint Connector_USB:USB_B_TE_5787834_Vertical -> Connector_JST:JST_XH_B5B-XH-A_1x05_P2.50mm_Vertical
- moved J5 58.2 mm to (184.0, 70.7), turned to -90 degrees
- moved J7 31.3 mm to (153.3, 39.9)
- moved J2 24.6 mm to (122.4, 47.7), turned to 30 degrees
- moved J3 24.5 mm to (109.2, 87.1), turned to 90 degrees
- moved J4 24.4 mm to (136.7, 118.3), turned to 150 degrees
- moved J6 24.4 mm to (190.9, 70.7), turned to -90 degrees
- moved J1 22.8 mm to (182.9, 50.0), turned to 150 degrees
Connections:
- J2 pad 1: +12V -> /TX1
- J2 pad 3: RTS1 -> /RX1
- J3 pad 1: +12V -> /TX2
- J3 pad 3: RTS2 -> /RX2
- J4 pad 1: +12V -> /TX3
- J4 pad 3: RTS3 -> /RX3
- J5 pad 1: +12V -> /TX4
- J5 pad 3: RTS4 -> /RX4
- J6 pad 1: +12V -> /TX5
- J6 pad 3: RTS5 -> /RX5
- J7 pad 1: Net-(J7-VBUS) -> /TX4
- J7 pad 2: DUP_N -> /RX4
- J7 pad 3: DUP_P -> /TX5
- J7 pad 4: GND -> /RX5
- J7 pad 5: /USB Hub/USB_SHEILD -> GND
Routing:
- net +3.3V: track 298.8 -> 0.00 mm, vias 18 -> 0
- net /TX3: track 0.00 -> 112.8 mm
- net /RX3: track 0.00 -> 103.5 mm
- net /TX2: track 0.00 -> 85.1 mm
- net /RX2: track 0.00 -> 80.3 mm
- net D2-: track 76.3 -> 0.00 mm, vias 1 -> 0
- net D2+: track 76.2 -> 0.00 mm, vias 1 -> 0
- net D3+: track 70.1 -> 0.00 mm
- net D3-: track 70.0 -> 0.00 mm
- net /TX4: track 0.00 -> 63.1 mm
- net D4-: track 56.1 -> 0.00 mm, vias 1 -> 0
- net D4+: track 56.0 -> 0.00 mm, vias 1 -> 0
- net /RX5: track 0.00 -> 49.0 mm
- net /RX4: track 0.00 -> 48.3 mm
- net D1-: track 47.6 -> 0.00 mm, vias 1 -> 0
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- removed copper zone on B.Cu, net /USB Hub/USB_SHEILD
- removed copper zone on F.Cu, net /USB Hub/USB_SHEILD
- removed copper zone on In1.Cu, net GND
- removed copper zone on In2.Cu, net GND
Other:
- copper layers 4 -> 2
- rule solder_mask_min_width: 0.1016 -> 0.12
- board text added: "https://github.com/daveismith/r2-warpcore-center-simple <<hash>>"
- board text removed: "0"
- board text removed: "1"
- board text removed: "2"
- board text removed: "CFG"
- board text removed: "https://github.com/daveismith/r2-warpcore-center <<hash>>"
