File: dome_center_pcb.kicad_sch (KiCad schematic)
At the start: 16 parts, among them J1 350211-1, J2 Conn_01x14_Pin, J3 Conn_01x14_Pin, J4 Conn_01x14_Pin, J5 Conn_01x14_Pin, J6 Conn_01x14_Pin, U10 DS2431P+T, U11 AMS1117-3.3, U6 DS2431P+T, U7 DS2431P+T, U8 DS2431P+T, U9 DS2431P+T

Commit message: Conversion to a simplified version.
Parts:
- removed C47, C50: 22uF, Capacitor_SMD:C_0805_2012Metric, symbol Device:C
- removed C48, C49: 10uF, Capacitor_SMD:C_0603_1608Metric, symbol Device:C
- removed J2, J3, J4, J5, J6: Conn_01x14_Pin, Connector_JST:JST_XH_B14B-XH-A_1x14_P2.50mm_Vertical, symbol Connector:Conn_01x14_Pin
- removed U10, U6, U7, U8, U9: DS2431P+T, easyeda2kicad:TSOC-6_L4.0-W4.0-P1.27-BL, symbol easyeda2kicad:DS2431P+T
- removed U11: AMS1117-3.3, Package_TO_SOT_SMD:SOT-223-3_TabPin2, symbol Regulator_Linear:AMS1117-3.3
- added J10, J11, J12, J8, J9: 171825-4, easyeda2kicad:HDR-TH_4P-P2.54-D1.0, symbol easyeda2kicad:171825-4
- added J13: Conn_01x07_Pin, Connector_JST:JST_XH_B7B-XH-A_1x07_P2.50mm_Vertical, symbol Connector:Conn_01x07_Pin
- added J2, J3, J4, J5, J6: Conn_01x03_Pin, Connector_JST:JST_XH_B3B-XH-A_1x03_P2.50mm_Vertical, symbol Connector:Conn_01x03_Pin
- added J7: Conn_01x05_Pin, Connector_JST:JST_XH_B5B-XH-A_1x05_P2.50mm_Vertical, symbol Connector:Conn_01x05_Pin
Connections:
- net +12V: now also J10.4, J11.4, J12.4, J8.4, J9.4
- net +5V: now also J10.1, J11.1, J12.1, J8.1, J9.1
- net GND: now also J10.2, J10.3, J11.2, J11.3, J12.2, J12.3, J13.7 (Pin_7), J2.2 (Pin_2), J3.2 (Pin_2), J4.2 (Pin_2), J5.2 (Pin_2), J6.2 (Pin_2), J7.5 (Pin_5), J8.2, J8.3, J9.2, J9.3
- new net RX1: J13.2 (Pin_2), J2.3 (Pin_3)
- new net RX2: J13.4 (Pin_4), J3.3 (Pin_3)
- new net RX3: J13.6 (Pin_6), J4.3 (Pin_3)
- new net RX4: J5.3 (Pin_3), J7.2 (Pin_2)
- new net RX5: J6.3 (Pin_3), J7.4 (Pin_4)
- new net TX1: J13.1 (Pin_1), J2.1 (Pin_1)
- new net TX2: J13.3 (Pin_3), J3.1 (Pin_1)
- new net TX3: J13.5 (Pin_5), J4.1 (Pin_1)
- new net TX4: J5.1 (Pin_1), J7.1 (Pin_1)
- new net TX5: J6.1 (Pin_1), J7.3 (Pin_3)
- no-connect marks 20 -> 0
Other:
- removed sheet FTDI
- removed sheet USB Hub
