File: ftdi.kicad_sch (KiCad schematic)
At the start: 48 parts, among them U1 FT4232H, U3 FT2232HL, U4 93LC56BT-I/OT, U5 93LC56BT-I/OT, X1 X322512MSB4SI, X2 X322512MSB4SI

Commit message: Conversion to a simplified version.
Parts:
- removed C1, C18, C39, C41, C43, C45: 4.7uF, Resistor_SMD:R_0402_1005Metric, symbol Device:C
- removed C10, C11, C12, C13, C14, C15, C16, C17, C2, C3, C4, C5, C6, C7, C8, C9: 100nF, Capacitor_SMD:C_0402_1005Metric, symbol Device:C
- removed C35, C36, C37, C38: 33pF, Resistor_SMD:R_0201_0603Metric, symbol Device:C
- removed C40, C42, C44, C46: 100nF, Resistor_SMD:R_0402_1005Metric, symbol Device:C
- removed FB1, FB2, FB3, FB4: 600Ω@100MHz, Resistor_SMD:R_0603_1608Metric, symbol Device:FerriteBead_Small
- removed R1, R8: 12K, Resistor_SMD:R_0402_1005Metric, symbol Device:R
- removed R2, R7: 1K, Resistor_SMD:R_0402_1005Metric, symbol Device:R
- removed R3, R5: 2K, Resistor_SMD:R_0402_1005Metric, symbol Device:R
- removed R4, R6: 10K, Resistor_SMD:R_0402_1005Metric, symbol Device:R
- removed U1: FT4232H, Package_QFP:LQFP-64_10x10mm_P0.5mm, symbol Interface_USB:FT4232H
- removed U3: FT2232HL, easyeda2kicad:LQFP-64_L10.0-W10.0-P0.50-LS12.0-TL, symbol easyeda2kicad:FT2232HL
- removed U4, U5: 93LC56BT-I/OT, easyeda2kicad:SOT-23-6_L2.9-W1.6-P0.95-LS2.8-BR, symbol easyeda2kicad:93LC56BT-I_OT
- removed X1, X2: X322512MSB4SI, easyeda2kicad:OSC-SMD_4P-L3.2-W2.5-BL, symbol easyeda2kicad:X322512MSB4SI
Connections:
- no-connect marks 35 -> 0
Other:
- note removed: "VCCIO Decoupling"
